File: KiCad/Tiny_Marquee.kicad_pcb (KiCad board)
At the start: 2 copper layers, 140 x 45 mm, 70 parts, among them J1 ADC6, J2 ADC7, J3 12 V, J4 5 V, J5 GND, J6 Barrel_Jack, Q1 FDN337N, Q2 FDN337N, Q3 FDN337N, Q4 FDN337N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

Commit message: Update to v0.3, switching C5 to 10uF, 35 V.
Parts:
- C5: value 100uF -> 10uF
Other:
- board text added: "MiniMarquee v0.3"
- board text removed: "MiniMarquee v0.2"
