File: KiCad/Tiny_Marquee.sch (KiCad schematic (older format))
At the start: 70 parts, among them J1 ADC6, J2 ADC7, J3 12 V, J4 5 V, J5 GND, J6 Barrel_Jack, Q1 FDN337N, Q2 FDN337N, Q3 FDN337N, Q4 FDN337N, Q5 FDN337N, Q6 FDN337N, U1 ATMEGA168-20AU, U2 AMS1117-5V, Y1 16MHz

Commit message: Update to v0.3, switching C5 to 10uF, 35 V.
Parts:
- C1, C2, C3, C4: symbol Device:C_Small -> Tiny_Marquee-rescue:C_Small-Device
- C5: value 100uF -> 10uF; symbol Device:CP1_Small -> Tiny_Marquee-rescue:CP1_Small-Device
- C6: symbol Device:CP1_Small -> Tiny_Marquee-rescue:CP1_Small-Device
- H1, H2, H3, H4, H5, H6, H7: symbol Mechanical:MountingHole -> Tiny_Marquee-rescue:MountingHole-Mechanical
- J6: symbol Connector:Barrel_Jack_Switch -> Tiny_Marquee-rescue:Barrel_Jack_Switch-Connector
- R1, R10, R11, R12, R13, R2, R3, R4, R5, R6, R7, R8, R9, RV_1, RV_10, RV_11, RV_12, RV_2, RV_3, RV_4, RV_5, RV_6, RV_7, RV_8, RV_9: symbol Device:R -> Tiny_Marquee-rescue:R-Device
- Y1: symbol Device:Crystal_Small -> Tiny_Marquee-rescue:Crystal_Small-Device
Changed lines of the file:
@@
 EESchema Schematic File Version 4
-LIBS:Tiny_Marquee-cache
-EELAYER 26 0
+EELAYER 30 0
 EELAYER END
 $Descr A4 11693 8268
@@
 $EndComp
 $Comp
-L power:GND #PWR021
+L Tiny_Marquee-rescue:GND-power #PWR021
 U 1 1 5BB4F8CF
 P 9800 6000
@@
 $EndComp
 $Comp
-L power:+12V #PWR020
+L Tiny_Marquee-rescue:+12V-power #PWR020
 U 1 1 5BB4F98D
 P 7700 1100
@@
 $EndComp
 $Comp
-L Device:R RV_4
+L Tiny_Marquee-rescue:R-Device RV_4
 U 1 1 5BB4FB2A
 P 9550 4250
@@
 $EndComp
 $Comp
-L Device:R RV_8
+L Tiny_Marquee-rescue:R-Device RV_8
 U 1 1 5BB4FC65
 P 9550 4050
@@
 $EndComp
 $Comp
-L Device:R RV_12
+L Tiny_Marquee-rescue:R-Device RV_12
 U 1 1 5BB4FCA8
 P 9550 3850
@@
 $EndComp
 $Comp
-L Device:R RV_11
+L Tiny_Marquee-rescue:R-Device RV_11
 U 1 1 5BB50BF5
 P 9550 3000
@@
 $EndComp
 $Comp
-L Device:R RV_7
+L Tiny_Marquee-rescue:R-Device RV_7
 U 1 1 5BB50C5B
 P 9550 3200
@@
 $EndComp
 $Comp
-L Device:R RV_3
+L Tiny_Marquee-rescue:R-Device RV_3
 U 1 1 5BB50CA2
 P 9550 3400
@@
 $EndComp
 $Comp
-L power:+5V #PWR05
+L Tiny_Marquee-rescue:+5V-power #PWR05
 U 1 1 5BB51CF5
 P 1200 900
@@
 $EndComp
 $Comp
-L power:GND #PWR07
+L Tiny_Marquee-rescue:GND-power #PWR07
 U 1 1 5BB51EED
 P 1200 3350
@@
 $EndComp
 $Comp
-L Device:C_Small C2
+L Tiny_Marquee-rescue:C_Small-Device C2
 U 1 1 5BB521EA
 P 1200 1750
@@
 $EndComp
 $Comp
-L power:GND #PWR06
+L Tiny_Marquee-rescue:GND-power #PWR06
 U 1 1 5BB5232A
 P 1200 1950
@@
 $EndComp
 $Comp
-L Device:Crystal_Small Y1
+L Tiny_Marquee-rescue:Crystal_Small-Device Y1
 U 1 1 5BB52662
 P 3900 1650
@@
 $EndComp
 $Comp
-L Device:C_Small C3
+L Tiny_Marquee-rescue:C_Small-Device C3
 U 1 1 5BB52B6C
 P 3750 1800
@@
 $EndComp
 $Comp
-L Device:C_Small C4
+L Tiny_Marquee-rescue:C_Small-Device C4
 U 1 1 5BB52BD6
 P 4050 1800
@@
 $EndComp
 $Comp
-L power:GND #PWR011
+L Tiny_Marquee-rescue:GND-power #PWR011
 U 1 1 5BB52EC7
 P 3900 1950
@@
 $EndComp
 $Comp
-L power:GND #PWR012
+L Tiny_Marquee-rescue:GND-power #PWR012
 U 1 1 5BB53211
 P 4050 5550
@@
 $EndComp
 $Comp
-L Device:R R1
+L Tiny_Marquee-rescue:R-Device R1
 U 1 1 5BB533B0
 P 3400 4800
@@
 $EndComp
 $Comp
-L power:+5V #PWR08
+L Tiny_Marquee-rescue:+5V-power #PWR08
 U 1 1 5BB53CCC
 P 3400 4600
@@
 SCK
 $Comp
-L power:GND #PWR017
+L Tiny_Marquee-rescue:GND-power #PWR017
 U 1 1 5BB5779D
 P 6350 3100
@@
 $EndComp
 $Comp
-L power:+5V #PWR016
+L Tiny_Marquee-rescue:+5V-power #PWR016
 U 1 1 5BB57A2C
 P 6350 2800
@@
 SW1
 $Comp
-L power:GND #PWR015
+L Tiny_Marquee-rescue:GND-power #PWR015
 U 1 1 5BC3819C
 P 6050 6050
@@
 $EndComp
 $Comp
-L Device:R R2
+L Tiny_Marquee-rescue:R-Device R2
 U 1 1 5BC381A5
 P 5100 4800
@@
 $EndComp
 $Comp
-L Device:R R3
+L Tiny_Marquee-rescue:R-Device R3
 U 1 1 5BC381AB
 P 5100 5100
@@
 $EndComp
 $Comp
-L Device:R R4
+L Tiny_Marquee-rescue:R-Device R4
 U 1 1 5BC381B1
 P 5100 5400
@@
 $EndComp
 $Comp
-L power:+12V #PWR014
+L Tiny_Marquee-rescue:+12V-power #PWR014
 U 1 1 5BC3A6FC
 P 6050 4050
@@
 $EndComp
 $Comp
-L Device:R R7
+L Tiny_Marquee-rescue:R-Device R7
 U 1 1 5BC3E4CC
 P 5800 5650
@@
 $EndComp
 $Comp
-L Device:R R6
+L Tiny_Marquee-rescue:R-Device R6
 U 1 1 5BC3E5F0
 P 5600 5650
@@
 $EndComp
 $Comp
-L Device:R R5
+L Tiny_Marquee-rescue:R-Device R5
 U 1 1 5BC3E67D
 P 5400 5650
@@
 Power In
 $Comp
-L Connector:Barrel_Jack_Switch J6
+L Tiny_Marquee-rescue:Barrel_Jack_Switch-Connector J6
 U 1 1 5BC448AC
 P 5300 1350
@@
 Connection ~ 6300 1550
 $Comp
-L power:GND #PWR019
+L Tiny_Marquee-rescue:GND-power #PWR019
 U 1 1 5BC45AB5
 P 6700 1650
@@
 $EndComp
 $Comp
-L power:+5V #PWR018
+L Tiny_Marquee-rescue:+5V-power #PWR018
 U 1 1 5BC45BB0
 P 6700 1150
@@
 $EndComp
 $Comp
-L power:+12V #PWR013
+L Tiny_Marquee-rescue:+12V-power #PWR013
 U 1 1 5BC45C5B
 P 5850 1150
@@
 	5850 1150 5850 1250
 $Comp
-L Device:CP1_Small C6
+L Tiny_Marquee-rescue:CP1_Small-Device C6
 U 1 1 5BC4726C
 P 6700 1400
@@
 $EndComp
 $Comp
-L Device:CP1_Small C5
+L Tiny_Marquee-rescue:CP1_Small-Device C5
 U 1 1 5BC479E9
 P 5850 1400
 F 0 "C5" H 5860 1470 50  0000 L CNN
-F 1 "100uF" H 5900 1300 50  0000 L CNN
+F 1 "10uF" H 5900 1300 50  0000 L CNN
 F 2 "Capacitor_Tantalum_SMD:CP_EIA-7343-15_Kemet-W_Pad2.25x2.55mm_HandSolder" H 5850 1400 50  0001 C CNN
 F 3 "" H 5850 1400 50  0001 C CNN
@@
 Connection ~ 5850 1550
 $Comp
-L Device:C_Small C1
+L Tiny_Marquee-rescue:C_Small-Device C1
 U 1 1 5BC48E38
 P 1050 1250
@@
 	1050 1050 1050 1150
 $Comp
-L power:GND #PWR02
+L Tiny_Marquee-rescue:GND-power #PWR02
 U 1 1 5BC49190
 P 1050 1400
@@
 	3750 2750 3750 2800
 $Comp
-L power:GND #PWR010
+L Tiny_Marquee-rescue:GND-power #PWR010
 U 1 1 5BC4A1BC
 P 3750 2800
@@
 $EndComp
 $Comp
-L power:+5V #PWR09
+L Tiny_Marquee-rescue:+5V-power #PWR09
 U 1 1 5BC4A2CF
 P 3750 2400
@@
 $EndComp
 $Comp
-L power:+5V #PWR01
+L Tiny_Marquee-rescue:+5V-power #PWR01
 U 1 1 5BC4CE33
 P 950 4100
@@
 $EndComp
 $Comp
-L power:+12V #PWR03
+L Tiny_Marquee-rescue:+12V-power #PWR03
 U 1 1 5BC4D072
 P 1150 4100
@@
 	950  4300 950  4100
 $Comp
-L power:GND #PWR04
+L Tiny_Marquee-rescue:GND-power #PWR04
 U 1 1 5BC4DA70
 P 1150 4500
@@
 $EndComp
 $Comp
-L Device:R R13
+L Tiny_Marquee-rescue:R-Device R13
 U 1 1 5C746083
 P 9550 5600
@@
 $EndComp
 $Comp
-L Device:R R12
+L Tiny_Marquee-rescue:R-Device R12
 U 1 1 5C76A52D
 P 9350 5600
@@
 $EndComp
 $Comp
-L Device:R R11
+L Tiny_Marquee-rescue:R-Device R11
 U 1 1 5C76A5AB
 P 9150 5600
@@
 $EndComp
 $Comp
-L Device:R R10
+L Tiny_Marquee-rescue:R-Device R10
 U 1 1 5C76A7FF
 P 8850 5350
@@
 	9150 4750 9150 5450
 $Comp
-L Device:R R9
+L Tiny_Marquee-rescue:R-Device R9
 U 1 1 5C78E467
 P 8850 5050
@@
 $EndComp
 $Comp
-L Device:R R8
+L Tiny_Marquee-rescue:R-Device R8
 U 1 1 5C78E4E7
 P 8850 4750
@@
 $EndComp
 $Comp
-L Device:R RV_2
+L Tiny_Marquee-rescue:R-Device RV_2
 U 1 1 5C880F06
 P 9550 2550
@@
 $EndComp
 $Comp
-L Device:R RV_6
+L Tiny_Marquee-rescue:R-Device RV_6
 U 1 1 5C880F0C
 P 9550 2350
@@
 $EndComp
 $Comp
-L Device:R RV_10
+L Tiny_Marquee-rescue:R-Device RV_10
 U 1 1 5C880F12
 P 9550 2150
@@
 $EndComp
 $Comp
-L Device:R RV_9
+L Tiny_Marquee-rescue:R-Device RV_9
 U 1 1 5C880F18
 P 9550 1300
@@
 $EndComp
 $Comp
-L Device:R RV_5
+L Tiny_Marquee-rescue:R-Device RV_5
 U 1 1 5C880F1E
 P 9550 1500
@@
 $EndComp
 $Comp
-L Device:R RV_1
+L Tiny_Marquee-rescue:R-Device RV_1
 U 1 1 5C880F24
 P 9550 1700
@@
 	2450 4800 500  4800
 $Comp
-L Mechanical:MountingHole H1
+L Tiny_Marquee-rescue:MountingHole-Mechanical H1
 U 1 1 5C6D9FF7
 P 700 5100
@@
 Mechanical
 $Comp
-L Mechanical:MountingHole H2
+L Tiny_Marquee-rescue:MountingHole-Mechanical H2
 U 1 1 5C704A92
 P 700 5350
@@
 $EndComp
 $Comp
-L Mechanical:MountingHole H3
+L Tiny_Marquee-rescue:MountingHole-Mechanical H3
 U 1 1 5C704B2A
 P 700 5600
@@
 $EndComp
 $Comp
-L Mechanical:MountingHole H4
+L Tiny_Marquee-rescue:MountingHole-Mechanical H4
 U 1 1 5C704BC4
 P 700 5850
@@
 $EndComp
 $Comp
-L Mechanical:MountingHole H5
+L Tiny_Marquee-rescue:MountingHole-Mechanical H5
 U 1 1 5C721EAC
 P 1600 5600
@@
 $EndComp
 $Comp
-L Mechanical:MountingHole H6
+L Tiny_Marquee-rescue:MountingHole-Mechanical H6
 U 1 1 5CB8B984
 P 1600 5100
@@
 $EndComp
 $Comp
-L Mechanical:MountingHole H7
+L Tiny_Marquee-rescue:MountingHole-Mechanical H7
 U 1 1 5CB8BA48
 P 1600 5350
